Commit message: created laser transform publisher

File: src/jackal/jackal_description/urdf/accessories.urdf.xacro (robot description, xacro)
@@ -19,6 +19,6 @@
                        topic="$(optenv JACKAL_LASER_TOPIC front/scan)"/>
     <joint name="$(optenv JACKAL_LASER_MOUNT front)_laser_mount_joint" type="fixed">
-      <origin xyz="$(optenv JACKAL_LASER_OFFSET 0 0 0)"
-              rpy="$(optenv JACKAL_LASER_RPY 0 0 0)" />
+      <origin xyz="$(optenv JACKAL_LASER_OFFSET 0 0 0.19)"
+              rpy="$(optenv JACKAL_LASER_RPY -3.14 0 0)" />
       <parent link="$(optenv JACKAL_LASER_MOUNT front)_mount" />
       <child link="$(optenv JACKAL_LASER_MOUNT front)_laser_mount" />

Commit message: better mapping/navigation

File: src/jackal/jackal_description/urdf/accessories.urdf.xacro (robot description, xacro)
@@ -19,5 +19,5 @@
                        topic="$(optenv JACKAL_LASER_TOPIC front/scan)"/>
     <joint name="$(optenv JACKAL_LASER_MOUNT front)_laser_mount_joint" type="fixed">
-      <origin xyz="$(optenv JACKAL_LASER_OFFSET 0 0 0.19)"
+      <origin xyz="$(optenv JACKAL_LASER_OFFSET 0 0 0.17)"
               rpy="$(optenv JACKAL_LASER_RPY -3.14 0 0)" />
       <parent link="$(optenv JACKAL_LASER_MOUNT front)_mount" />

Commit message: path planning for both robots/added camera and image processing

File: src/jackal/jackal_description/urdf/accessories.urdf.xacro (robot description, xacro)
@@ -8,4 +8,5 @@
     jackal_gazebo/launch/jackal_world.launch
     jackal_base/launch/base.launch
+  <xacro:include filename="accessories/kinect_camera.gazebo.xacro"/>
   -->
   <!-- Macros to generate standoffs for offset payload mounting. -->

File: src/jackal/jackal_description/urdf/accessories/sick_lms1xx_mount.urdf.xacro (robot description, xacro)
@@ -41,5 +41,5 @@
     <joint name="${prefix}_laser_joint" type="fixed">
       <!-- This offset is from the base of the bracket to the LIDAR's focal point. -->
-      <origin xyz="0 0 0.149" rpy="0 0 0" />
+      <origin xyz="0 0 0.05" rpy="-3.14 0 0" />
       <parent link="${prefix}_laser_mount" />
       <child link="${prefix}_laser" />

File: src/jackal/jackal_description/urdf/custom_example.urdf (robot description, URDF)
Before this commit: robot None, 0 links, 8 joints
Joints:
- removed joint rear_camera_bracket_joint
- removed joint rear_camera_mount_joint
- removed joint rear_laser_mount_joint
- removed joint rear_upper_camera_bracket_joint
- removed joint rear_upper_camera_mount_joint
- joint front_camera_bracket_joint: origin xyz=0.007 0 0.02450 rpy=0 0 0 -> xyz=0.05 0 -0.01 rpy=0 0 0
- joint front_laser_mount_joint: origin xyz=0 0 0.002 rpy=0 0 0 -> xyz=0 0 0 rpy=0 0 0

File: src/jackal/jackal_description/urdf/jackal.urdf.xacro (robot description, xacro)
@@ -172,5 +172,7 @@
        default each one to off.-->
   <xacro:include filename="accessories.urdf.xacro" />
-  <!-- Optional custom includes. -->
-  <!--<xacro:include filename="$(optenv JACKAL_URDF_EXTRAS empty.urdf)" />-->
+  <xacro:include filename="custom_example.urdf" />
+  <!-- Optional custom includes.
+  <xacro:include filename="$(optenv JACKAL_URDF_EXTRAS empty.urdf)" />
+-->
 </robot>
